File: backplane.kicad_sch (KiCad schematic)
At the start: 20 parts, among them J101 USB_C_Receptacle_USB2.0, SW101 RESET, U101 USB2514BI, Y101 24MHZ

Commit message: update board
Other:
- note added: "MECHANICAL"
- note added: "USB-IN"
- moved on the sheet: H101, H102, H103, H104, H105, H106, H107, H109, J101, R101, R102

Commit message: Auto-commit Fri Feb 17 13:50:17 EST 2023
Changed lines of the file:
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@@
     (pin "1")
   )
-  (sheet (at 30.48 135.89) (size 24.13 22.86) (fields_autoplaced)
+  (sheet (at 21.59 22.86) (size 24.13 22.86) (fields_autoplaced)
     (stroke (width 0.1524) (type solid) (color 0 0 0 0))
     (fill (color 0 0 0 0.0000))
-    (property "Sheet name" "PSU" (id 0) (at 30.48 135.1784 0)
+    (property "Sheet name" "PSU" (id 0) (at 21.59 22.1484 0)
       (effects (font (size 1.27 1.27)) (justify left bottom))
     )
-    (property "Sheet file" "powersupply.kicad_sch" (id 1) (at 30.48 159.3346 0)
+    (property "Sheet file" "powersupply.kicad_sch" (id 1) (at 21.59 46.3046 0)
       (effects (font (size 1.27 1.27)) (justify left top))
     )
   )
-  (sheet (at 78.74 135.89) (size 24.13 22.86) (fields_autoplaced)
+  (sheet (at 21.59 57.15) (size 24.13 22.86) (fields_autoplaced)
     (stroke (width 0.1524) (type solid) (color 0 0 0 0))
     (fill (color 0 0 0 0.0000))
-    (property "Sheet name" "SLOTS" (id 0) (at 78.74 135.1784 0)
+    (property "Sheet name" "SLOTS" (id 0) (at 21.59 56.4384 0)
       (effects (font (size 1.27 1.27)) (justify left bottom))
     )
-    (property "Sheet file" "expansionslots.kicad_sch" (id 1) (at 78.74 159.3346 0)
+    (property "Sheet file" "expansionslots.kicad_sch" (id 1) (at 21.59 80.5946 0)
       (effects (font (size 1.27 1.27)) (justify left top))
     )
   )
-  (sheet (at 123.19 134.62) (size 24.13 24.13) (fields_autoplaced)
+  (sheet (at 22.225 92.075) (size 24.13 24.13) (fields_autoplaced)
     (stroke (width 0.1524) (type solid) (color 0 0 0 0))
     (fill (color 0 0 0 0.0000))
-    (property "Sheet name" "AUX" (id 0) (at 123.19 133.9084 0)
+    (property "Sheet name" "AUX" (id 0) (at 22.225 91.3634 0)
       (effects (font (size 1.27 1.27)) (justify left bottom))
     )
-    (property "Sheet file" "aux.kicad_sch" (id 1) (at 123.19 159.3346 0)
+    (property "Sheet file" "aux.kicad_sch" (id 1) (at 22.225 116.7896 0)
       (effects (font (size 1.27 1.27)) (justify left top))
     )
